Commit message: tested fix for .stl scale problem in robot visualisation

File: src/ros/crustcrawler_smart_arm/smart_arm_description/urdf/smart_arm.xacro (robot description, xacro)
@@ -144,5 +144,5 @@
                 <origin xyz="0.0 0.0 0.005" rpy="0 0 0" />
                 <geometry>
-                    <mesh filename="package://smart_arm_description/meshes/collada/arm_shoulder_pan.dae"/>
+                    <mesh filename="package://smart_arm_description/meshes/arm_pan_1.stl"/>
                 </geometry>
                 <material name="Grey" />
@@ -151,5 +151,5 @@
                 <origin xyz="0.0 0.0 0.0" rpy="0 0 0" />
                 <geometry>
-                    <mesh filename="package://smart_arm_description/meshes/collada/arm_shoulder_pan.dae"/>
+                    <mesh filename="package://smart_arm_description/meshes/arm_pan_1.stl"/>
                 </geometry>
             </collision>
@@ -254,5 +254,5 @@
                 <origin xyz="0.0 0.0 0.0" rpy="0 0 0" />
                 <geometry>
-                    <mesh filename="package://smart_arm_description/meshes/collada/arm_left_finger.dae"/>
+                    <mesh filename="package://smart_arm_description/meshes/claw.stl"/>
                 </geometry>
                 <material name="Green" />
@@ -333,4 +333,8 @@
             <kd value="1.0" />
         </gazebo>
+	<gazebo reference="left_claw_link">
+            <material>SmartArm/GunMetalBrushedAluminum</material>
+            <turnGravityOff>true</turnGravityOff>
+        </gazebo>
         <gazebo reference="shoulder_pan_joint">
             <stopKd value="1.0" />
