Commit message: fixed error with arm_shoulder_pitch_link by reloading the arm_shoulder_pitch.stl file from its original source

File: src/ros/smart_arm_desc/smart_arm_desc.xacro (robot description, xacro)
@@ -58,10 +58,10 @@
 	<!-- Shoulder tilt joint -->
         <joint name="shoulder_pitch_joint" type="revolute">
-            <origin xyz="${0.077/1.414} 0 ${0.040 + 0.077/1.414}" rpy="0 0 0" />
+            <origin xyz="${0.077/1.414} 0 ${0.040 + 0.077/1.414}" rpy="0 -0.7854 0" />
             <parent link="arm_shoulder_pan_link"/>
             <child link="arm_shoulder_pitch_link" />
             <axis xyz="0 -1 0"/>
-            <limit  lower="-1.04719755" upper="1.972222" effort="300" velocity="1.17" />
-            <safety_controller k_position="100" k_velocity="15.0" soft_lower_limit="${-1.04719755+0.1}" soft_upper_limit="${1.972222-0.1}" />
+            <limit  lower="-2.007" upper="2.007" effort="300" velocity="1.17" />
+            <safety_controller k_position="100" k_velocity="15.0" soft_lower_limit="-2" soft_upper_limit="2" />
             <dynamics damping="50" friction="1"/>
         </joint>
@@ -111,5 +111,5 @@
 	<!-- Right finger joint -->
         <joint name="right_finger_joint" type="revolute">
-            <origin xyz="0.052 0 0.003" rpy="0 0 1.5708" />
+            <origin xyz="0.058 0 0.007" rpy="0 0 1.5708" />
             <parent link="arm_right_finger_link"/>
             <child link="arm_right_gripper_link" />
@@ -122,5 +122,5 @@
 	<!-- Left finger joint -->
         <joint name="left_finger_joint" type="revolute">
-            <origin xyz="0.052 0 0.003" rpy="0 0 -1.5708" />
+            <origin xyz="0.058 0 0.007" rpy="0 0 -1.5708" />
             <parent link="arm_left_finger_link"/>
             <child link="arm_left_gripper_link" />
@@ -133,9 +133,20 @@
 	<!-- Right connector joint -->
         <joint name="right_connector_joint" type="revolute">
-            <origin xyz="0.059 -0.005 -0.010" rpy="0 0 1.5708" />
+            <origin xyz="0.049 -0.005 -0.009" rpy="0 0 -1.5708" />
             <parent link="arm_wrist_roll_link"/>
             <child link="arm_right_connector_link" />
+            <axis xyz="0 0 1"/>
+	    <mimic joint="claw_joint" multiplier="1"/>
+            <!-- From -14 to 45 degrees -->
+            <limit  lower="-0.2618" upper="0.9599" effort="300" velocity="1.17" />
+            <dynamics damping="50" friction="1"/>
+        </joint>
+	<!-- Left connector joint -->
+        <joint name="left_connector_joint" type="revolute">
+            <origin xyz="0.049 0.005 -0.009" rpy="0 0 1.5708" />
+            <parent link="arm_wrist_roll_link"/>
+            <child link="arm_left_connector_link" />
+            <axis xyz="0 0 1"/>
 	    <mimic joint="claw_joint" multiplier="-1"/>
-            <axis xyz="0 0 1"/>
             <!-- From -14 to 45 degrees -->
             <limit  lower="-0.9599" upper="0.2618" effort="300" velocity="1.17" />
@@ -322,5 +333,5 @@
             <inertial>
                 <mass value="0.0225" />
-                <origin xyz="${-0.01*0.5-0.004*0.866} ${-0.005*0.866-0.004*0.5} 0.014" rpy="3.1415 -0 0.139" />
+                <origin xyz="${-0.01*0.5-0.004*0.866} ${0.005*0.866+0.004*0.5} 0.014" rpy="3.1415 -0 0.139" />
                 <inertia ixx="1.0" ixy="0.0" ixz="0.0"
                          iyy="1.0" iyz="0.0"
@@ -342,4 +353,26 @@
         </link>
 <link name="arm_right_connector_link">
+            <inertial>
+                <mass value="0.0225" />
+                <origin xyz="${-0.01*0.5-0.004*0.866} ${-0.005*0.866-0.004*0.5} 0.014" rpy="0 0 0" />
+                <inertia ixx="1.0" ixy="0.0" ixz="0.0"
+                         iyy="1.0" iyz="0.0"
+                         izz="1.0" />
+            </inertial>
+            <visual>
+                <origin xyz="-0.005 -0.005 0" rpy="0 0 0" />
+                <geometry>
+                    <mesh filename="package://smart_arm_desc/meshes/arm_connector.stl"/>
+                </geometry>
+                <material name="matArm" />
+            </visual>
+            <collision>
+                <origin xyz="0.005 0.005 0" rpy="0 0 0" />
+                <geometry>
+                    <mesh filename="package://smart_arm_desc/meshes/arm_connector.stl"/>
+                </geometry>
+            </collision>
+        </link>
+<link name="arm_left_connector_link">
             <inertial>
                 <mass value="0.0225" />
